Commit message: component checking

File: fix.urdf (robot description, URDF)
Before this commit: robot sda10f, 22 links, 21 joints
Links:
- link arm_left_link_1_s: geometry collision mesh filename=package://sda10f_description/meshes/sda10f/collision/motoma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; visual mesh filename=package://sda10f_description/meshes/sda10f/visual/motoman_a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
- link arm_left_link_2_l: geometry collision mesh filename=package://sda10f_description/meshes/sda10f/collision/motoma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; visual mesh filename=package://sda10f_description/meshes/sda10f/visual/motoman_a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
- link arm_left_link_3_e: geometry collision mesh filename=package://sda10f_description/meshes/sda10f/collision/motoma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; visual mesh filename=package://sda10f_description/meshes/sda10f/visual/motoman_a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
- link arm_left_link_4_u: geometry collision mesh filename=package://sda10f_description/meshes/sda10f/collision/motoma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; visual mesh filename=package://sda10f_description/meshes/sda10f/visual/motoman_a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
- link arm_left_link_5_r: geometry collision mesh filename=package://sda10f_description/meshes/sda10f/collision/motoma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; visual mesh filename=package://sda10f_description/meshes/sda10f/visual/motoman_a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
- link arm_left_link_6_b: geometry collision mesh filename=package://sda10f_description/meshes/sda10f/collision/motoma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; visual mesh filename=package://sda10f_description/meshes/sda10f/visual/motoman_a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
- link arm_left_link_7_t: geometry collision mesh filename=package://sda10f_description/meshes/sda10f/collision/motoma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; visual mesh filename=package://sda10f_description/meshes/sda10f/visual/motoman_a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
- link arm_right_link_1_s: geometry collision mesh filename=package://sda10f_description/meshes/sda10f/collision/motoma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; visual mesh filename=package://sda10f_description/meshes/sda10f/visual/motoman_a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
- link arm_right_link_2_l: geometry collision mesh filename=package://sda10f_description/meshes/sda10f/collision/motoma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; visual mesh filename=package://sda10f_description/meshes/sda10f/visual/motoman_a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
- link arm_right_link_3_e: geometry collision mesh filename=package://sda10f_description/meshes/sda10f/collision/motoma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; visual mesh filename=package://sda10f_description/meshes/sda10f/visual/motoman_a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
- link arm_right_link_4_u: geometry collision mesh filename=package://sda10f_description/meshes/sda10f/collision/motoma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; visual mesh filename=package://sda10f_description/meshes/sda10f/visual/motoman_a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
- link arm_right_link_5_r: geometry collision mesh filename=package://sda10f_description/meshes/sda10f/collision/motoma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; visual mesh filename=package://sda10f_description/meshes/sda10f/visual/motoman_a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
- link arm_right_link_6_b: geometry collision mesh filename=package://sda10f_description/meshes/sda10f/collision/motoma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; visual mesh filename=package://sda10f_description/meshes/sda10f/visual/motoman_a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
- link arm_right_link_7_t: geometry collision mesh filename=package://sda10f_description/meshes/sda10f/collision/motoma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; visual mesh filename=package://sda10f_description/meshes/sda10f/visual/motoman_a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
- link base_link: geometry collision mesh filename=package://sda10f_description/meshes/sda10f/collision/motoma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; visual mesh filename=package://sda10f_description/meshes/sda10f/visual/motoman_b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
- link motoman_left_hand: geometry collision mesh filename=package://sda10f_description/meshes/sda10f/collision/vacuum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; visual mesh filename=package://sda10f_description/meshes/sda10f/visual/vacuum_gr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
- link motoman_right_hand: geometry collision mesh filename=package://sda10f_description/meshes/sda10f/collision/modelO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; visual mesh filename=package://sda10f_description/meshes/sda10f/visual/modelO42.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
- link torso_link: geometry collision mesh filename=package://sda10f_description/meshes/sda10f/collision/motoma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; visual mesh filename=package://sda10f_description/meshes/sda10f/visual/motoman_a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
